File: KiCAD/Detector de particulas (FISICA III).kicad_pcb (KiCad board)
At the start: 2 copper layers, 27 parts, among them J1 Conn_01x02_Female, J2 Conn_01x02_Female, J3 Conn_01x02_Pin, J4 Conn_01x02_Pin, J5 Conn_01x02_Pin, U1 OPA2134PA

Commit message: nuevo pcb completo
Parts:
- removed the C1 at (124.5, 57.5)
- removed the C2 at (120.5, 55.0)
- removed the C3 at (20.9, 7.38)
- removed the C4 at (132.8, 48.5)
- removed the C5 at (142.0, 48.5)
- removed the C6 at (156.5, 63.5)
- removed the C7 at (131.5, 66.5)
- removed the C8 at (158.0, 55.2)
- removed the C9 at (150.8, 56.0)
- removed the D1 at (86.0, 65.5)
- removed the D2 at (93.8, 65.5)
- removed the D3 at (101.8, 65.5)
- removed the D4 at (109.8, 65.5)
- removed the J1 at (27.3, 13.6)
- removed the J2 at (165.8, 67.0)
- removed the J3 at (12.9, 36.8)
- removed the J4 at (17.6, 36.8)
- removed the J5 at (146.5, 56.0)
- removed the R1 at (122.8, 70.3)
- removed the R2 at (127.8, 62.7)
- removed the R3 at (128.8, 55.0)
- removed the R4 at (156.0, 48.5)
- removed the R5 at (146.5, 70.5)
- removed the R6 at (142.2, 71.8)
- removed the R7 at (142.2, 67.8)
- removed the R8 at (151.2, 63.0)
- removed the U1 at (134.6, 54.9)
- added C1: 10p, Capacitor_THT:C_Disc_D3.0mm_W1.6mm_P2.50mm, F.Cu at (69.0, 206.5)
- added C1: 10p, Capacitor_THT:C_Disc_D3.0mm_W1.6mm_P2.50mm, F.Cu at (155.5, 203.5)
- added C1: 10p, Capacitor_THT:C_Disc_D3.0mm_W1.6mm_P2.50mm, F.Cu at (154.5, 72.0)
- added C1: 10p, Capacitor_THT:C_Disc_D3.0mm_W1.6mm_P2.50mm, F.Cu at (69.5, 73.1)
- added C2: 10p, Capacitor_THT:C_Disc_D3.0mm_W1.6mm_P2.50mm, F.Cu at (66.5, 210.5)
- added C2: 10p, Capacitor_THT:C_Disc_D3.0mm_W1.6mm_P2.50mm, F.Cu at (152.0, 76.0)
- added C2: 10p, Capacitor_THT:C_Disc_D3.0mm_W1.6mm_P2.50mm, F.Cu at (67.0, 77.1)
- added C2: 10p, Capacitor_THT:C_Disc_D3.0mm_W1.6mm_P2.50mm, F.Cu at (153.0, 207.5)
- added C3: 100n, Capacitor_THT:C_Disc_D3.0mm_W1.6mm_P2.50mm, F.Cu at (76.0, 213.0)
- added C3: 100n, Capacitor_THT:C_Disc_D3.0mm_W1.6mm_P2.50mm, F.Cu at (161.5, 78.5)
- added C3: 100n, Capacitor_THT:C_Disc_D3.0mm_W1.6mm_P2.50mm, F.Cu at (162.5, 210.0)
- added C3: 100n, Capacitor_THT:C_Disc_D3.0mm_W1.6mm_P2.50mm, F.Cu at (76.5, 79.6)
- added C4: 100n, Capacitor_THT:C_Disc_D3.0mm_W1.6mm_P2.50mm, F.Cu at (145.0, 64.2)
- added C4: 100n, Capacitor_THT:C_Disc_D3.0mm_W1.6mm_P2.50mm, F.Cu at (146.0, 195.8)
- added C4: 100n, Capacitor_THT:C_Disc_D3.0mm_W1.6mm_P2.50mm, F.Cu at (59.5, 198.8)
- added C4: 100n, Capacitor_THT:C_Disc_D3.0mm_W1.6mm_P2.50mm, F.Cu at (60.0, 65.4)
- added C5: 100n, Capacitor_THT:C_Disc_D3.0mm_W1.6mm_P2.50mm, F.Cu at (145.0, 55.0)
- added C5: 100n, Capacitor_THT:C_Disc_D3.0mm_W1.6mm_P2.50mm, F.Cu at (60.0, 56.1)
- added C5: 100n, Capacitor_THT:C_Disc_D3.0mm_W1.6mm_P2.50mm, F.Cu at (146.0, 186.5)
- added C5: 100n, Capacitor_THT:C_Disc_D3.0mm_W1.6mm_P2.50mm, F.Cu at (59.5, 189.5)
- added C6: 10p, Capacitor_THT:C_Disc_D3.0mm_W1.6mm_P2.50mm, F.Cu at (79.0, 38.1)
- added C6: 10p, Capacitor_THT:C_Disc_D3.0mm_W1.6mm_P2.50mm, F.Cu at (78.5, 171.5)
- added C6: 10p, Capacitor_THT:C_Disc_D3.0mm_W1.6mm_P2.50mm, F.Cu at (165.0, 168.5)
- added C6: 10p, Capacitor_THT:C_Disc_D3.0mm_W1.6mm_P2.50mm, F.Cu at (164.0, 37.0)
- added C7: 100n, Capacitor_THT:C_Disc_D3.0mm_W1.6mm_P2.50mm, F.Cu at (77.5, 200.0)
- added C7: 100n, Capacitor_THT:C_Disc_D3.0mm_W1.6mm_P2.50mm, F.Cu at (163.0, 65.5)
- added C7: 100n, Capacitor_THT:C_Disc_D3.0mm_W1.6mm_P2.50mm, F.Cu at (78.0, 66.6)
- added C7: 100n, Capacitor_THT:C_Disc_D3.0mm_W1.6mm_P2.50mm, F.Cu at (164.0, 197.0)
- added C8: 47u, Capacitor_THT:CP_Radial_D6.3mm_P2.50mm, F.Cu at (152.8, 170.5)
- added C8: 47u, Capacitor_THT:CP_Radial_D6.3mm_P2.50mm, F.Cu at (66.8, 40.1)
- added C8: 47u, Capacitor_THT:CP_Radial_D6.3mm_P2.50mm, F.Cu at (66.2, 173.5)
- added C8: 47u, Capacitor_THT:CP_Radial_D6.3mm_P2.50mm, F.Cu at (151.8, 39.0)
- added C9: 100n, Capacitor_THT:C_Disc_D3.0mm_W1.6mm_P2.50mm, F.Cu at (152.5, 46.2)
- added C9: 100n, Capacitor_THT:C_Disc_D3.0mm_W1.6mm_P2.50mm, F.Cu at (67.5, 47.4)
- added C9: 100n, Capacitor_THT:C_Disc_D3.0mm_W1.6mm_P2.50mm, F.Cu at (67.0, 180.8)
- added C9: 100n, Capacitor_THT:C_Disc_D3.0mm_W1.6mm_P2.50mm, F.Cu at (153.5, 177.8)
- added D1: BPW34, OptoDevice:Osram_BPW34S-SMD, B.Cu at (161.8, 85.0)
- added D1: BPW34, OptoDevice:Osram_BPW34S-SMD, B.Cu at (162.8, 216.5)
- added D1: BPW34, OptoDevice:Osram_BPW34S-SMD, B.Cu at (76.3, 219.5)
- added D1: BPW34, OptoDevice:Osram_BPW34S-SMD, B.Cu at (76.8, 86.1)
- added D2: BPW34, OptoDevice:Osram_BPW34S-SMD, B.Cu at (76.3, 227.2)
- added D2: BPW34, OptoDevice:Osram_BPW34S-SMD, B.Cu at (161.8, 92.8)
- added D2: BPW34, OptoDevice:Osram_BPW34S-SMD, B.Cu at (76.8, 93.9)
- added D2: BPW34, OptoDevice:Osram_BPW34S-SMD, B.Cu at (162.8, 224.2)
- added D3: BPW34, OptoDevice:Osram_BPW34S-SMD, B.Cu at (76.3, 235.2)
- added D3: BPW34, OptoDevice:Osram_BPW34S-SMD, B.Cu at (76.8, 101.9)
- added D3: BPW34, OptoDevice:Osram_BPW34S-SMD, B.Cu at (162.8, 232.2)
- added D3: BPW34, OptoDevice:Osram_BPW34S-SMD, B.Cu at (161.8, 100.8)
- added D4: BPW34, OptoDevice:Osram_BPW34S-SMD, B.Cu at (76.8, 109.9)
- added D4: BPW34, OptoDevice:Osram_BPW34S-SMD, B.Cu at (162.8, 240.2)
- added D4: BPW34, OptoDevice:Osram_BPW34S-SMD, B.Cu at (76.3, 243.2)
- added D4: BPW34, OptoDevice:Osram_BPW34S-SMD, B.Cu at (161.8, 108.8)
- added J1: Conn_01x02_Female, Connector_PinHeader_2.54mm:PinHeader_1x02_P2.54mm_Vertical, F.Cu at (153.0, 31.2)
- added J1: Conn_01x02_Female, Connector_PinHeader_2.54mm:PinHeader_1x02_P2.54mm_Vertical, F.Cu at (67.5, 165.8)
- added J1: Conn_01x02_Female, Connector_PinHeader_2.54mm:PinHeader_1x02_P2.54mm_Vertical, F.Cu at (68.0, 32.4)
- added J1: Conn_01x02_Female, Connector_PinHeader_2.54mm:PinHeader_1x02_P2.54mm_Vertical, F.Cu at (154.0, 162.8)
- added J2: Conn_01x02_Female, Connector_PinHeader_2.54mm:PinHeader_1x02_P2.54mm_Vertical, F.Cu at (164.5, 162.8)
- added J2: Conn_01x02_Female, Connector_PinHeader_2.54mm:PinHeader_1x02_P2.54mm_Vertical, F.Cu at (78.5, 32.4)
- added J2: Conn_01x02_Female, Connector_PinHeader_2.54mm:PinHeader_1x02_P2.54mm_Vertical, F.Cu at (163.5, 31.2)
- added J2: Conn_01x02_Female, Connector_PinHeader_2.54mm:PinHeader_1x02_P2.54mm_Vertical, F.Cu at (78.0, 165.8)
- added J3: Conn_01x02_Pin, Connector_PinHeader_2.54mm:PinHeader_1x02_P2.54mm_Vertical, F.Cu at (155.2, 213.7)
- added J3: Conn_01x02_Pin, Connector_PinHeader_2.54mm:PinHeader_1x02_P2.54mm_Vertical, F.Cu at (69.2, 83.3)
- added J3: Conn_01x02_Pin, Connector_PinHeader_2.54mm:PinHeader_1x02_P2.54mm_Vertical, F.Cu at (68.8, 216.7)
- added J3: Conn_01x02_Pin, Connector_PinHeader_2.54mm:PinHeader_1x02_P2.54mm_Vertical, F.Cu at (154.2, 82.2)
- added J4: Conn_01x02_Pin, Connector_PinHeader_2.54mm:PinHeader_1x02_P2.54mm_Vertical, F.Cu at (60.5, 165.5)
- added J4: Conn_01x02_Pin, Connector_PinHeader_2.54mm:PinHeader_1x02_P2.54mm_Vertical, F.Cu at (61.0, 32.1)
- added J4: Conn_01x02_Pin, Connector_PinHeader_2.54mm:PinHeader_1x02_P2.54mm_Vertical, F.Cu at (146.0, 31.0)
- added J4: Conn_01x02_Pin, Connector_PinHeader_2.54mm:PinHeader_1x02_P2.54mm_Vertical, F.Cu at (147.0, 162.5)
- added J5: Conn_01x02_Pin, Connector_PinHeader_2.54mm:PinHeader_1x02_P2.54mm_Vertical, F.Cu at (67.5, 51.6)
- added J5: Conn_01x02_Pin, Connector_PinHeader_2.54mm:PinHeader_1x02_P2.54mm_Vertical, F.Cu at (67.0, 185.0)
- added J5: Conn_01x02_Pin, Connector_PinHeader_2.54mm:PinHeader_1x02_P2.54mm_Vertical, F.Cu at (152.5, 50.5)
- added J5: Conn_01x02_Pin, Connector_PinHeader_2.54mm:PinHeader_1x02_P2.54mm_Vertical, F.Cu at (153.5, 182.0)
- added R1: 4k7, Resistor_THT:R_Axial_DIN0207_L6.3mm_D2.5mm_P7.62mm_Horizontal, F.Cu at (81.8, 75.4)
- added R1: 4k7, Resistor_THT:R_Axial_DIN0207_L6.3mm_D2.5mm_P7.62mm_Horizontal, F.Cu at (167.8, 205.8)
- added R1: 4k7, Resistor_THT:R_Axial_DIN0207_L6.3mm_D2.5mm_P7.62mm_Horizontal, F.Cu at (166.8, 74.2)
- added R1: 4k7, Resistor_THT:R_Axial_DIN0207_L6.3mm_D2.5mm_P7.62mm_Horizontal, F.Cu at (81.3, 208.8)
- added R2: 15k, Resistor_THT:R_Axial_DIN0207_L6.3mm_D2.5mm_P7.62mm_Horizontal, F.Cu at (159.2, 69.2)
- added R2: 15k, Resistor_THT:R_Axial_DIN0207_L6.3mm_D2.5mm_P7.62mm_Horizontal, F.Cu at (74.2, 70.4)
- added R2: 15k, Resistor_THT:R_Axial_DIN0207_L6.3mm_D2.5mm_P7.62mm_Horizontal, F.Cu at (160.2, 200.8)
- added R2: 15k, Resistor_THT:R_Axial_DIN0207_L6.3mm_D2.5mm_P7.62mm_Horizontal, F.Cu at (73.7, 203.8)
- added R3: 10M, Resistor_THT:R_Axial_DIN0309_L9.0mm_D3.2mm_P2.54mm_Vertical, F.Cu at (66.5, 202.2)
- added R3: 10M, Resistor_THT:R_Axial_DIN0309_L9.0mm_D3.2mm_P2.54mm_Vertical, F.Cu at (67.0, 68.9)
- added R3: 10M, Resistor_THT:R_Axial_DIN0309_L9.0mm_D3.2mm_P2.54mm_Vertical, F.Cu at (152.0, 67.8)
- added R3: 10M, Resistor_THT:R_Axial_DIN0309_L9.0mm_D3.2mm_P2.54mm_Vertical, F.Cu at (153.0, 199.2)
- added R4: 1k, Resistor_THT:R_Axial_DIN0207_L6.3mm_D2.5mm_P7.62mm_Horizontal, F.Cu at (60.0, 42.1)
- added R4: 1k, Resistor_THT:R_Axial_DIN0207_L6.3mm_D2.5mm_P7.62mm_Horizontal, F.Cu at (59.5, 175.5)
- added R4: 1k, Resistor_THT:R_Axial_DIN0207_L6.3mm_D2.5mm_P7.62mm_Horizontal, F.Cu at (146.0, 172.5)
- added R4: 1k, Resistor_THT:R_Axial_DIN0207_L6.3mm_D2.5mm_P7.62mm_Horizontal, F.Cu at (145.0, 41.0)
- added R5: 100k, Resistor_THT:R_Axial_DIN0207_L6.3mm_D2.5mm_P7.62mm_Horizontal, F.Cu at (163.5, 182.3)
- added R5: 100k, Resistor_THT:R_Axial_DIN0207_L6.3mm_D2.5mm_P7.62mm_Horizontal, F.Cu at (77.5, 51.9)
- added R5: 100k, Resistor_THT:R_Axial_DIN0207_L6.3mm_D2.5mm_P7.62mm_Horizontal, F.Cu at (77.0, 185.3)
- added R5: 100k, Resistor_THT:R_Axial_DIN0207_L6.3mm_D2.5mm_P7.62mm_Horizontal, F.Cu at (162.5, 50.8)
- added R6: 10k, Resistor_THT:R_Axial_DIN0207_L6.3mm_D2.5mm_P7.62mm_Horizontal, F.Cu at (169.3, 186.2)
- added R6: 10k, Resistor_THT:R_Axial_DIN0207_L6.3mm_D2.5mm_P7.62mm_Horizontal, F.Cu at (82.8, 189.2)
- added R6: 10k, Resistor_THT:R_Axial_DIN0207_L6.3mm_D2.5mm_P7.62mm_Horizontal, F.Cu at (168.3, 54.8)
- added R6: 10k, Resistor_THT:R_Axial_DIN0207_L6.3mm_D2.5mm_P7.62mm_Horizontal, F.Cu at (83.3, 55.9)
- added R7: 10k, Resistor_THT:R_Axial_DIN0207_L6.3mm_D2.5mm_P7.62mm_Horizontal, F.Cu at (165.5, 193.8)
- added R7: 10k, Resistor_THT:R_Axial_DIN0207_L6.3mm_D2.5mm_P7.62mm_Horizontal, F.Cu at (79.5, 63.4)
- added R7: 10k, Resistor_THT:R_Axial_DIN0207_L6.3mm_D2.5mm_P7.62mm_Horizontal, F.Cu at (79.0, 196.8)
- added R7: 10k, Resistor_THT:R_Axial_DIN0207_L6.3mm_D2.5mm_P7.62mm_Horizontal, F.Cu at (164.5, 62.3)
- added R8: 2k2, Resistor_THT:R_Axial_DIN0207_L6.3mm_D2.5mm_P7.62mm_Horizontal, F.Cu at (71.9, 174.5)
- added R8: 2k2, Resistor_THT:R_Axial_DIN0207_L6.3mm_D2.5mm_P7.62mm_Horizontal, F.Cu at (72.4, 41.1)
- added R8: 2k2, Resistor_THT:R_Axial_DIN0207_L6.3mm_D2.5mm_P7.62mm_Horizontal, F.Cu at (158.4, 171.5)
- added R8: 2k2, Resistor_THT:R_Axial_DIN0207_L6.3mm_D2.5mm_P7.62mm_Horizontal, F.Cu at (157.4, 40.0)
- added U1: OPA2134PA, Package_DIP:DIP-8_W7.62mm, F.Cu at (65.9, 196.9)
- added U1: OPA2134PA, Package_DIP:DIP-8_W7.62mm, F.Cu at (152.4, 193.9)
- added U1: OPA2134PA, Package_DIP:DIP-8_W7.62mm, F.Cu at (151.4, 62.4)
- added U1: OPA2134PA, Package_DIP:DIP-8_W7.62mm, F.Cu at (66.4, 63.5)
Routing:
- net +9V: track 0.00 -> 608.8 mm
- net Net-(U1-In2-): track 0.00 -> 316.4 mm
- net Net-(U1-Out1): track 0.00 -> 146.9 mm
- net Net-(D1-K): track 0.00 -> 114.0 mm
- net Net-(J5-Pin_2): track 0.00 -> 109.0 mm
- net Net-(J3-Pin_1): track 0.00 -> 86.8 mm
- net /Output: track 0.00 -> 86.3 mm
- net Net-(U1-In1+): track 0.00 -> 75.2 mm
- net Net-(C4-Pad2): track 0.00 -> 72.5 mm
- net Net-(U1-In2+): track 0.00 -> 69.9 mm
- net Net-(J1-Pin_1): track 0.00 -> 28.3 mm
- net Net-(J5-Pin_1): track 0.00 -> 17.1 mm
- net Net-(C1-Pad2): track 0.00 -> 16.0 mm
- added copper zone on B.Cu, net GND
Other:
- board outline added: 124.5 x 226 mm

Commit message: primera version terminada
Parts:
- removed the C1 at (69.0, 206.5)
- removed the C1 at (155.5, 203.5)
- removed the C1 at (154.5, 72.0)
- removed the C1 at (69.5, 73.1)
- removed the C2 at (66.5, 210.5)
- removed the C2 at (152.0, 76.0)
- removed the C2 at (67.0, 77.1)
- removed the C2 at (153.0, 207.5)
- removed the C3 at (76.0, 213.0)
- removed the C3 at (161.5, 78.5)
- removed the C3 at (162.5, 210.0)
- removed the C3 at (76.5, 79.6)
- removed the C4 at (145.0, 64.2)
- removed the C4 at (146.0, 195.8)
- removed the C4 at (59.5, 198.8)
- removed the C4 at (60.0, 65.4)
- removed the C5 at (145.0, 55.0)
- removed the C5 at (60.0, 56.1)
- removed the C5 at (146.0, 186.5)
- removed the C5 at (59.5, 189.5)
- removed the C6 at (79.0, 38.1)
- removed the C6 at (78.5, 171.5)
- removed the C6 at (165.0, 168.5)
- removed the C6 at (164.0, 37.0)
- removed the C7 at (77.5, 200.0)
- removed the C7 at (163.0, 65.5)
- removed the C7 at (78.0, 66.6)
- removed the C7 at (164.0, 197.0)
- removed the C8 at (152.8, 170.5)
- removed the C8 at (66.8, 40.1)
- removed the C8 at (66.2, 173.5)
- removed the C8 at (151.8, 39.0)
- removed C9 (x4): 100n, Capacitor_THT:C_Disc_D3.0mm_W1.6mm_P2.50mm
- removed the D1 at (161.8, 85.0)
- removed the D1 at (162.8, 216.5)
- removed the D1 at (76.3, 219.5)
- removed the D1 at (76.8, 86.1)
- removed the D2 at (76.3, 227.2)
- removed the D2 at (161.8, 92.8)
- removed the D2 at (76.8, 93.9)
- removed the D2 at (162.8, 224.2)
- removed the D3 at (76.3, 235.2)
- removed the D3 at (76.8, 101.9)
- removed the D3 at (162.8, 232.2)
- removed the D3 at (161.8, 100.8)
- removed the D4 at (76.8, 109.9)
- removed the D4 at (162.8, 240.2)
- removed the D4 at (76.3, 243.2)
- removed the D4 at (161.8, 108.8)
- removed the J1 at (153.0, 31.2)
- removed the J1 at (67.5, 165.8)
- removed the J1 at (68.0, 32.4)
- removed the J1 at (154.0, 162.8)
- removed the J2 at (164.5, 162.8)
- removed the J2 at (78.5, 32.4)
- removed the J2 at (163.5, 31.2)
- removed the J2 at (78.0, 165.8)
- removed J3 (x4), J4 (x4), J5 (x4): Conn_01x02_Pin, Connector_PinHeader_2.54mm:PinHeader_1x02_P2.54mm_Vertical
- removed the R1 at (81.8, 75.4)
- removed the R1 at (167.8, 205.8)
- removed the R1 at (166.8, 74.2)
- removed the R1 at (81.3, 208.8)
- removed the R2 at (159.2, 69.2)
- removed the R2 at (74.2, 70.4)
- removed the R2 at (160.2, 200.8)
- removed the R2 at (73.7, 203.8)
- removed the R3 at (66.5, 202.2)
- removed the R3 at (67.0, 68.9)
- removed the R3 at (152.0, 67.8)
- removed the R3 at (153.0, 199.2)
- removed the R4 at (60.0, 42.1)
- removed the R4 at (59.5, 175.5)
- removed the R4 at (146.0, 172.5)
- removed the R4 at (145.0, 41.0)
- removed the R5 at (163.5, 182.3)
- removed the R5 at (77.5, 51.9)
- removed the R5 at (77.0, 185.3)
- removed the R5 at (162.5, 50.8)
- removed the R6 at (169.3, 186.2)
- removed the R6 at (82.8, 189.2)
- removed the R6 at (168.3, 54.8)
- removed the R6 at (83.3, 55.9)
- removed the R7 at (165.5, 193.8)
- removed the R7 at (79.5, 63.4)
- removed the R7 at (79.0, 196.8)
- removed the R7 at (164.5, 62.3)
- removed R8 (x4): 2k2, Resistor_THT:R_Axial_DIN0207_L6.3mm_D2.5mm_P7.62mm_Horizontal
- removed the U1 at (65.9, 196.9)
- removed the U1 at (152.4, 193.9)
- removed the U1 at (151.4, 62.4)
- removed the U1 at (66.4, 63.5)
- added C1: 10p, Capacitor_THT:C_Disc_D3.0mm_W1.6mm_P2.50mm, F.Cu at (131.0, 58.5)
- added C2: 10p, Capacitor_THT:C_Disc_D3.0mm_W1.6mm_P2.50mm, F.Cu at (137.4, 58.5)
- added C3: 100n, Capacitor_THT:C_Disc_D3.0mm_W1.6mm_P2.50mm, F.Cu at (130.7, 72.9)
- added C4: 100n, Capacitor_THT:C_Disc_D3.0mm_W1.6mm_P2.50mm, F.Cu at (156.2, 58.5)
- added C5: 100n, Capacitor_THT:C_Disc_D3.0mm_W1.6mm_P2.50mm, F.Cu at (167.9, 61.9)
- added C6: 10p, Capacitor_THT:C_Disc_D3.0mm_W1.6mm_P2.50mm, F.Cu at (167.9, 69.5)
- added C7: 100n, Capacitor_THT:C_Disc_D3.0mm_W1.6mm_P2.50mm, F.Cu at (183.7, 62.4)
- added C8: 47u, Capacitor_THT:CP_Radial_D6.3mm_P2.50mm, F.Cu at (175.3, 60.6)
- added D1: BPW34, OptoDevice:Osram_BPW34S-SMD, B.Cu at (150.3, 65.3)
- added D2: BPW34, OptoDevice:Osram_BPW34S-SMD, B.Cu at (143.9, 65.3)
- added D3: BPW34, OptoDevice:Osram_BPW34S-SMD, B.Cu at (137.3, 65.3)
- added D4: BPW34, OptoDevice:Osram_BPW34S-SMD, B.Cu at (131.1, 65.3)
- added J1: Conn_01x02_Female, Connector_PinHeader_2.54mm:PinHeader_1x02_P2.54mm_Vertical, F.Cu at (186.8, 60.1)
- added J2: Conn_01x02_Female, Connector_PinHeader_2.54mm:PinHeader_1x02_P2.54mm_Vertical, F.Cu at (186.6, 69.9)
- added R1: 4k7, Resistor_THT:R_Axial_DIN0207_L6.3mm_D2.5mm_P7.62mm_Horizontal, F.Cu at (141.9, 72.5)
- added R2: 15k, Resistor_THT:R_Axial_DIN0207_L6.3mm_D2.5mm_P7.62mm_Horizontal, F.Cu at (152.9, 72.5)
- added R3: 10M, Resistor_THT:R_Axial_DIN0204_L3.6mm_D1.6mm_P7.62mm_Horizontal, F.Cu at (151.7, 58.5)
- added R4: 1k, Resistor_THT:R_Axial_DIN0207_L6.3mm_D2.5mm_P7.62mm_Horizontal, F.Cu at (170.1, 58.5)
- added R5: 100k, Resistor_THT:R_Axial_DIN0207_L6.3mm_D2.5mm_P7.62mm_Horizontal, F.Cu at (172.1, 73.1)
- added R6: 10k, Resistor_THT:R_Axial_DIN0207_L6.3mm_D2.5mm_P7.62mm_Horizontal, F.Cu at (180.3, 65.3)
- added R7: 10k, Resistor_THT:R_Axial_DIN0207_L6.3mm_D2.5mm_P7.62mm_Horizontal, F.Cu at (175.9, 73.1)
- added U1: OPA2134PA, Package_DIP:DIP-8_W7.62mm, F.Cu at (156.3, 64.2)
Routing:
- net +9V: track 608.8 -> 114.7 mm
- net Net-(U1-In2-): track 316.4 -> 20.1 mm
- net Net-(U1-Out1): track 146.9 -> 24.6 mm
- net Net-(J5-Pin_2): track 109.0 -> 0.00 mm
- net Net-(J3-Pin_1): track 86.8 -> 0.00 mm
- net Net-(C4-Pad2): track 72.5 -> 3.78 mm
- net Net-(D1-K): track 114.0 -> 47.7 mm
- net /Output: track 86.3 -> 41.5 mm
- net Net-(U1-In1+): track 75.2 -> 31.0 mm
- net Net-(U1-In2+): track 69.9 -> 31.0 mm
- net Net-(J1-Pin_1): track 28.3 -> 0.00 mm
- net Net-(J5-Pin_1): track 17.1 -> 0.00 mm
- net Net-(C1-Pad2): track 16.0 -> 3.95 mm
Other:
- board size 124.5 x 226 mm -> 66 x 21.7 mm

Commit message: nuevo pcb
Parts:
- added C9: 100n, Capacitor_THT:C_Disc_D3.0mm_W1.6mm_P2.50mm, F.Cu at (150.8, 56.0)
- added J3: Conn_01x02_Pin, Connector_PinHeader_2.54mm:PinHeader_1x02_P2.54mm_Vertical, F.Cu at (12.9, 36.8)
- added J4: Conn_01x02_Pin, Connector_PinHeader_2.54mm:PinHeader_1x02_P2.54mm_Vertical, F.Cu at (17.6, 36.8)
- added J5: Conn_01x02_Pin, Connector_PinHeader_2.54mm:PinHeader_1x02_P2.54mm_Vertical, F.Cu at (146.5, 56.0)
- added R8: 2k2, Resistor_THT:R_Axial_DIN0207_L6.3mm_D2.5mm_P7.62mm_Horizontal, F.Cu at (151.2, 63.0)
- D1, D2, D3, D4: moved to F.Cu
- R3: footprint Resistor_THT:R_Axial_DIN0204_L3.6mm_D1.6mm_P7.62mm_Horizontal -> Resistor_THT:R_Axial_DIN0309_L9.0mm_D3.2mm_P2.54mm_Vertical
- moved J1 166.1 mm to (27.3, 13.6)
- moved C3 127.9 mm to (20.9, 7.38), turned to 0 degrees
- moved D1 64.3 mm to (86.0, 65.5), turned to 90 degrees
- moved C7 52.4 mm to (131.5, 66.5)
- moved D2 50.2 mm to (93.8, 65.5), turned to 90 degrees
- moved R6 38.6 mm to (142.2, 71.8), turned to 180 degrees
- moved D3 35.6 mm to (101.8, 65.5), turned to 90 degrees
- moved R7 34.1 mm to (142.2, 67.8), turned to 180 degrees
- moved C5 29.1 mm to (142.0, 48.5), turned to 0 degrees
- moved R2 27.0 mm to (127.8, 62.7), turned to -90 degrees
- moved R5 25.7 mm to (146.5, 70.5)
- moved C4 25.5 mm to (132.8, 48.5)
- moved U1 23.6 mm to (134.6, 54.9)
- moved R3 23.2 mm to (128.8, 55.0), turned to -90 degrees
- moved D4 21.4 mm to (109.8, 65.5), turned to 90 degrees
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Connections:
- C1 pad 1: Net-(D1-K) -> Net-(J3-Pin_1)
- C6 pad 2: /Output -> Net-(J5-Pin_2)
- J1 pad 1: +9V -> Net-(J1-Pin_1)
- R3 pad 2: Net-(D1-K) -> Net-(J3-Pin_1)
- R5 pad 1: /Output -> Net-(J5-Pin_2)
- U1 pad 2: Net-(D1-K) -> Net-(J3-Pin_1)
- U1 pad 7: /Output -> Net-(J5-Pin_2)
Routing:
- net +9V: track 114.7 -> 0.00 mm
- net Net-(D1-K): track 47.7 -> 0.00 mm
- net /Output: track 41.5 -> 0.00 mm
- net Net-(U1-In1+): track 31.0 -> 0.00 mm
- net Net-(U1-In2+): track 31.0 -> 0.00 mm
- net Net-(U1-Out1): track 24.6 -> 0.00 mm
- net Net-(U1-In2-): track 20.1 -> 0.00 mm
- net Net-(C1-Pad2): track 3.95 -> 0.00 mm
- net Net-(C4-Pad2): track 3.78 -> 0.00 mm
- removed copper zone on B.Cu, net GND
Other:
- board outline removed
